Commit message: working version on lab machine

File: EZGripper/ezgripper_driver/urdf/ezgripper_dual_articulated.urdf.xacro (robot description, xacro)
@@ -1,6 +1,6 @@
 <?xml version="1.0" encoding="UTF-8"?>
-<robot name="ezgripper" xmlns:xacro="http://www.ros.org/wiki/xacro">
+<robot name="ezgripper" xmlns:xacro="http://ros.org/wiki/xacro">
 <!--macro name="ezgripper" params="*origin"-->
-<macro name="ezgripper_dual" params="prefix parent_link *origin">
+<xacro:macro name="ezgripper_dual" params="prefix parent_link *origin">
     <!-- links -->
     <link name="${prefix}_ezgripper_palm_link">
@@ -40,6 +40,6 @@
     <ezgripper_knuckle_trans prefix="${prefix}" postfix="2"/>
     <gazebo_knuckle_jsp prefix="${prefix}" />
-</macro>
-<macro name="ezgripper_finger_L1" params="prefix postfix reflect">
+</xacro:macro>
+<xacro:macro name="ezgripper_finger_L1" params="prefix postfix reflect">
     <link name="${prefix}_ezgripper_finger_L1_${postfix}">
       <visual>
@@ -60,6 +60,6 @@
       </inertial>
     </link>
-</macro>
-<macro name="ezgripper_finger_L2" params="prefix postfix reflect">
+</xacro:macro>
+<xacro:macro name="ezgripper_finger_L2" params="prefix postfix reflect">
     <link name="${prefix}_ezgripper_finger_L2_${postfix}">
       <visual>
@@ -80,7 +80,7 @@
       </inertial>
     </link>
-</macro>
+</xacro:macro>
     <!-- joints -->
-<macro name="ezgripper_knuckle_palm_L1" params="prefix postfix reflectY reflectZ reflectR mimic_test">
+<xacro:macro name="ezgripper_knuckle_palm_L1" params="prefix postfix reflectY reflectZ reflectR mimic_test">
     <joint name="${prefix}_ezgripper_knuckle_palm_L1_${postfix}" type="revolute">
       <parent link="${prefix}_ezgripper_palm_link"/>
@@ -93,6 +93,6 @@
       </xacro:if>
     </joint>
-</macro>
-<macro name="ezgripper_knuckle_L1_L2" params="prefix postfix reflectY reflectZ reflectR mimic_test">
+</xacro:macro>
+<xacro:macro name="ezgripper_knuckle_L1_L2" params="prefix postfix reflectY reflectZ reflectR mimic_test">
     <joint name="${prefix}_ezgripper_knuckle_L1_L2_${postfix}" type="revolute">
       <parent link="${prefix}_ezgripper_finger_L1_${postfix}"/>
@@ -105,7 +105,7 @@
       </xacro:if>
     </joint>
-</macro>
+</xacro:macro>
     <!-- transmissions for Gazebo -->
-<macro name="ezgripper_knuckle_trans" params="prefix postfix">
+<xacro:macro name="ezgripper_knuckle_trans" params="prefix postfix">
    <transmission name="${prefix}_ezgripper_trans_${postfix}">
       <type>transmission_interface/SimpleTransmission</type>
@@ -118,6 +118,6 @@
       </actuator>
    </transmission>
-</macro>
-<macro name="gazebo_knuckle_jsp" params="prefix">
+</xacro:macro>
+<xacro:macro name="gazebo_knuckle_jsp" params="prefix">
    <gazebo>
      <plugin name="joint_state_publisher" filename="libgazebo_ros_joint_state_publisher.so">
@@ -125,5 +125,5 @@
      </plugin>
    </gazebo>
-</macro>
+</xacro:macro>
 <gazebo>
    <plugin name="gazebo_ros_control" filename="libgazebo_ros_control.so">

File: EZGripper/ezgripper_driver/urdf/ezgripper_dual_gen2.urdf.xacro (robot description, xacro)
@@ -1,6 +1,6 @@
 <?xml version="1.0" encoding="UTF-8"?>
-<robot name="ezgripper" xmlns:xacro="http://www.ros.org/wiki/xacro">
+<robot name="ezgripper" xmlns:xacro="http://ros.org/wiki/xacro">
 <!--macro name="ezgripper" params="*origin"-->
-<macro name="ezgripper_dual_gen2" params="prefix parent_link *origin">
+<xacro:macro name="ezgripper_dual_gen2" params="prefix parent_link *origin">
     <!-- links -->
     <link name="${prefix}_ezgripper_palm_link">
@@ -36,6 +36,6 @@
     <ezgripper_knuckle_trans prefix="${prefix}" postfix="2"/>
     <gazebo_knuckle_jsp prefix="${prefix}" />
-</macro>
-<macro name="ezgripper_finger" params="prefix postfix reflect">
+</xacro:macro>
+<xacro:macro name="ezgripper_finger" params="prefix postfix reflect">
     <link name="${prefix}_ezgripper_finger_${postfix}">
       <visual>
@@ -56,7 +56,7 @@
       </inertial>
     </link>
-</macro>
+</xacro:macro>
     <!-- joints -->
-<macro name="ezgripper_knuckle" params="prefix postfix reflectY reflectZ reflectR mimic_test">
+<xacro:macro name="ezgripper_knuckle" params="prefix postfix reflectY reflectZ reflectR mimic_test">
     <joint name="${prefix}_ezgripper_knuckle_${postfix}" type="revolute">
       <parent link="${prefix}_ezgripper_palm_link"/>
@@ -69,7 +69,7 @@
       </xacro:if>
     </joint>
-</macro>
+</xacro:macro>
     <!-- transmissions for Gazebo -->
-<macro name="ezgripper_knuckle_trans" params="prefix postfix">
+<xacro:macro name="ezgripper_knuckle_trans" params="prefix postfix">
    <transmission name="${prefix}_ezgripper_trans_${postfix}">
       <type>transmission_interface/SimpleTransmission</type>
@@ -82,6 +82,6 @@
       </actuator>
    </transmission>
-</macro>
-<macro name="gazeobo_knuckle_jsp" params="prefix">
+</xacro:macro>
+<xacro:macro name="gazeobo_knuckle_jsp" params="prefix">
    <gazebo>
      <plugin name="joint_state_publisher" filename="libgazebo_ros_joint_state_publisher.so">
@@ -89,5 +89,5 @@
      </plugin>
    </gazebo>
-</macro>
+</xacro:macro>
 <gazebo>
    <plugin name="gazebo_ros_control" filename="libgazebo_ros_control.so">

File: EZGripper/ezgripper_driver/urdf/ezgripper_dual_gen2_standalone.urdf.xacro (robot description, xacro)
@@ -1,8 +1,8 @@
 <?xml version="1.0" encoding="UTF-8"?>
-<robot name="ezgripper_stand_alone" xmlns:xacro="http://www.ros.org/wiki/xacro">
-<property name="ezgripper_offset_x" value="0.049"/>
-<property name="ezgripper_offset_y" value="0.0"/>
-<property name="ezgripper_offset_z" value="0.21"/>
-<xacro:include filename="$(find ezgripper_driver)/urdf/ezgripper_dual.urdf.xacro"/>
+<robot name="ezgripper_stand_alone" xmlns:xacro="http://ros.org/wiki/xacro">
+<xacro:property name="ezgripper_offset_x" value="0.0"/>
+<xacro:property name="ezgripper_offset_y" value="0.0"/>
+<xacro:property name="ezgripper_offset_z" value="0.0"/>
+<xacro:include filename="$(find ezgripper_driver)/urdf/ezgripper_dual_gen2_articulated.urdf.xacro"/>
 <!-- Add the gripper -->
 <ezgripper_dual prefix="left" parent_link="base_link">
@@ -19,5 +19,5 @@
            <cylinder length="0.42" radius="0.02"/>
         </geometry>
-        <origin rpy="0 0 0" xyz="0 0 0.21"/>
+        <origin rpy="0 0 0" xyz="0 0 0.0"/>
         <material name="red"/>
     </visual>

File: EZGripper/ezgripper_driver/urdf/ezgripper_dual_standalone.urdf.xacro (robot description, xacro)
@@ -1,8 +1,8 @@
 <?xml version="1.0" encoding="UTF-8"?>
-<robot name="ezgripper_stand_alone" xmlns:xacro="http://www.ros.org/wiki/xacro">
-<property name="ezgripper_offset_x" value="0.0"/>
-<property name="ezgripper_offset_y" value="0.0"/>
-<property name="ezgripper_offset_z" value="0.0"/>
-<xacro:include filename="$(find ezgripper_driver)/urdf/ezgripper_dual_gen2_articulated.urdf.xacro"/>
+<robot name="ezgripper_stand_alone" xmlns:xacro="http://ros.org/wiki/xacro">
+<xacro:property name="ezgripper_offset_x" value="0.049"/>
+<xacro:property name="ezgripper_offset_y" value="0.0"/>
+<xacro:property name="ezgripper_offset_z" value="0.21"/>
+<xacro:include filename="$(find ezgripper_driver)/urdf/ezgripper_dual.urdf.xacro"/>
 <!-- Add the gripper -->
 <ezgripper_dual prefix="left" parent_link="base_link">
@@ -12,14 +12,14 @@
 <joint name="fixed" type="fixed">
   <parent link="world"/>
-  <!--<child link="base_link"/>-->
+  <child link="base_link"/>
 </joint>
-<!--<link name="base_link">
+<link name="base_link">
    <visual>
        <geometry>
            <cylinder length="0.42" radius="0.02"/>
         </geometry>
-        <origin rpy="0 0 0" xyz="0 0 0.0"/>
+        <origin rpy="0 0 0" xyz="0 0 0.21"/>
         <material name="red"/>
     </visual>
-</link>-->
+</link>
 </robot>

File: EZGripper/ezgripper_driver/urdf/ezgripper_quad.urdf.xacro (robot description, xacro)
@@ -1,5 +1,5 @@
 <?xml version="1.0" encoding="UTF-8"?>
-<robot name="ezgripper" xmlns:xacro="http://www.ros.org/wiki/xacro">
-<macro name="ezgripper_quad" params="prefix parent_link *origin">
+<robot name="ezgripper" xmlns:xacro="http://ros.org/wiki/xacro">
+<xacro:macro name="ezgripper_quad" params="prefix parent_link *origin">
     <!-- links -->
     <link name="${prefix}_ezgripper_palm_link">
@@ -41,6 +41,6 @@
     <ezgripper_knuckle_trans prefix="${prefix}" postfix="4"/>
     <gazebo_knuckle_jsp prefix="${prefix}" />
-</macro>
-<macro name="ezgripper_finger" params="prefix postfix reflect">
+</xacro:macro>
+<xacro:macro name="ezgripper_finger" params="prefix postfix reflect">
     <link name="${prefix}_ezgripper_finger_${postfix}">
       <visual>
@@ -61,7 +61,7 @@
       </inertial>
     </link>
-</macro>
+</xacro:macro>
     <!-- joints -->
-<macro name="ezgripper_knuckle" params="prefix postfix reflectY reflectZ reflectR mimic_test">
+<xacro:macro name="ezgripper_knuckle" params="prefix postfix reflectY reflectZ reflectR mimic_test">
     <joint name="${prefix}_ezgripper_knuckle_${postfix}" type="revolute">
       <parent link="${prefix}_ezgripper_palm_link"/>
@@ -74,7 +74,7 @@
       </xacro:if>
     </joint>
-</macro>
+</xacro:macro>
     <!-- transmissions for Gazebo -->
-<macro name="ezgripper_knuckle_trans" params="prefix postfix">
+<xacro:macro name="ezgripper_knuckle_trans" params="prefix postfix">
    <transmission name="${prefix}_ezgripper_trans_${postfix}">
       <type>transmission_interface/SimpleTransmission</type>
@@ -87,6 +87,6 @@
       </actuator>
    </transmission>
-</macro>
-<macro name="gazebo_knuckle_jsp" params="prefix">
+</xacro:macro>
+<xacro:macro name="gazebo_knuckle_jsp" params="prefix">
     <gazebo>
       <plugin name="joint_state_publisher" filename="libgazebo_ros_joint_state_publisher.so">
@@ -94,5 +94,5 @@
       </plugin>
     </gazebo>
-</macro>
+</xacro:macro>
 <gazebo>
    <plugin name="gazebo_ros_control" filename="libgazebo_ros_control.so">

File: EZGripper/ezgripper_driver/urdf/ezgripper_quad_standalone.urdf.xacro (robot description, xacro)
@@ -1,12 +1,12 @@
 <?xml version="1.0" encoding="UTF-8"?>
-<robot name="ezgripper_stand_alone" xmlns:xacro="http://www.ros.org/wiki/xacro">
-<property name="ezgripper_offset_x" value="0.0"/>
-<property name="ezgripper_offset_y" value="0.0"/>
-<property name="ezgripper_offset_z" value="0.0"/>
-<xacro:include filename="$(find ezgripper_driver)/urdf/ezgripper_dual_gen2_articulated.urdf.xacro"/>
+<robot name="ezgripper_stand_alone" xmlns:xacro="http://ros.org/wiki/xacro">
+<xacro:property name="ezgripper_offset_x" value="0.049"/>
+<xacro:property name="ezgripper_offset_y" value="0.0"/>
+<xacro:property name="ezgripper_offset_z" value="0.21"/>
+<xacro:include filename="$(find ezgripper_driver)/urdf/ezgripper_quad.urdf.xacro"/>
 <!-- Add the gripper -->
-<ezgripper_dual prefix="left" parent_link="base_link">
+<ezgripper_quad prefix="left" parent_link="base_link">
 <origin xyz="${ezgripper_offset_x} ${ezgripper_offset_y} ${ezgripper_offset_z}" rpy="0 0 0"/>
-</ezgripper_dual>
+</ezgripper_quad>
 <link name="world"/>
 <joint name="fixed" type="fixed">
@@ -19,5 +19,5 @@
            <cylinder length="0.42" radius="0.02"/>
         </geometry>
-        <origin rpy="0 0 0" xyz="0 0 0.0"/>
+        <origin rpy="0 0 0" xyz="0 0 0.21"/>
         <material name="red"/>
     </visual>
